Commit message: clean up + arm_control pkg

File: src/arm_urdf/urdf/arm_control.xacro (robot description, xacro)
@@ -15,4 +15,5 @@
             </transmission>
         </xacro:macro>
+        <xacro:arm_control transmission="${prefix}_tran_0" joint="${prefix}_base_fixed_base_joint" motor="${prefix}_motor_0"/>
         <xacro:arm_control transmission="${prefix}_tran_1" joint="${prefix}_base_bridge_joint" motor="${prefix}_motor_1"/>
         <xacro:arm_control transmission="${prefix}_tran_2" joint="${prefix}_bridge_housing_joint" motor="${prefix}_motor_2"/>

File: src/arm_urdf/urdf/arm_gazebo.xacro (robot description, xacro)
@@ -1,4 +1,3 @@
 <?xml version='1.0' encoding='utf-8'?>
-<!-- panda.gazebo.xacro -->
 <robot xmlns:xacro="http://www.ros.org/wiki/xacro">
     <xacro:macro name="arm_gazebo_setting" params="prefix">
@@ -9,4 +8,5 @@
             </gazebo>
         </xacro:macro>
+        <xacro:arm_gazebo link="${prefix}_base_fixed"/>
         <xacro:arm_gazebo link="${prefix}_base"/>
         <xacro:arm_gazebo link="${prefix}_bridge"/>

File: src/arm_urdf/urdf/arm_urdf.xacro (robot description, xacro)
@@ -3,4 +3,10 @@
     <xacro:macro name="arm" params="prefix">
         <!-- links -->
+        <link name="${prefix}_base_fixed">
+            <inertial>
+            <mass value="0.5"/>
+            <inertia ixx="0.4" ixy="0.0" ixz="0.0" iyy="0.4" iyz="0.0" izz="0.2"/>
+            </inertial>
+        </link>
         <link name="${prefix}_base">
             <visual>
@@ -113,4 +119,12 @@
         <!-- joints -->
         <!-- joint names defined like so: ${prefix}_<parent>-<child>_joint -->
+        <joint name="${prefix}_base_fixed_base_joint" type="revolute">
+            <origin rpy="0.0 0 0" xyz="0.0 0 0"/>
+            <axis xyz="0 0 1"/>
+            <limit effort="1000.0" lower="${radians(-180)}" upper="${radians(180)}" velocity="0.5"/>
+            <parent link="${prefix}_base_fixed" />
+            <child link="${prefix}_base" />
+            <dynamics D="1" K="7000" mu_coulomb="0" mu_viscous="16" damping="0.003" friction="0.0"/>
+        </joint>
         <joint name="${prefix}_base_bridge_joint" type="revolute">
             <origin rpy="0.0 0 0" xyz="0.0 0 0.165"/>

File: src/arm_urdf/urdf/main.xacro (robot description, xacro)
@@ -14,5 +14,5 @@
     <joint name="base" type="fixed">
         <parent link="world" />
-        <child link="arm1_base" />
+        <child link="arm1_base_fixed" />
     </joint>
     <!-- NOTE: order of execution of above xacro does not matter -->

Commit message: + Pedistal and rgb camera

File: src/arm_urdf/urdf/arm_control.xacro (robot description, xacro)
@@ -1,4 +1,3 @@
 <?xml version="1.0"?>
-<!-- panda.control.xacro -->
 <robot xmlns:xacro="http://www.ros.org/wiki/xacro">
     <xacro:macro name="arm_control_setting" params="prefix">
@@ -20,7 +19,4 @@
         <xacro:arm_control transmission="${prefix}_tran_3" joint="${prefix}_housing_wrist_link_joint" motor="${prefix}_motor_3"/>
         <xacro:arm_control transmission="${prefix}_tran_4" joint="${prefix}_wrist_link_wrist_cuff_joint" motor="${prefix}_motor_4"/>
-        <gazebo>
-            <plugin name="gazebo_ros_control" filename="libgazebo_ros_control.so"/>
-        </gazebo>
     </xacro:macro>
 </robot>

File: src/arm_urdf/urdf/arm_gazebo.xacro (robot description, xacro)
@@ -14,4 +14,46 @@
         <xacro:arm_gazebo link="${prefix}_wrist_link"/>
         <xacro:arm_gazebo link="${prefix}_wrist_cuff"/>
+        <gazebo>
+            <plugin name="gazebo_ros_control" filename="libgazebo_ros_control.so"/>
+        </gazebo>
+        <gazebo reference="${prefix}_camera">
+            <sensor type="camera" name="camera1">
+            <update_rate>30.0</update_rate>
+            <camera name="head">
+                <horizontal_fov>1.3962634</horizontal_fov>
+                <image>
+                <width>800</width>
+                <height>800</height>
+                <format>R8G8B8</format>
+                </image>
+                <clip>
+                <near>0.02</near>
+                <far>300</far>
+                </clip>
+                <noise>
+                <type>gaussian</type>
+                <!-- Noise is sampled independently per pixel on each frame.
+                    That pixel's noise value is added to each of its color
+                    channels, which at that point lie in the range [0,1]. -->
+                <mean>0.0</mean>
+                <stddev>0.007</stddev>
+                </noise>
+            </camera>
+            <plugin name="camera_controller" filename="libgazebo_ros_camera.so">
+                <alwaysOn>true</alwaysOn>
+                <updateRate>0.0</updateRate>
+                <cameraName>bot/camera1</cameraName>
+                <imageTopicName>image_raw</imageTopicName>
+                <cameraInfoTopicName>camera_info</cameraInfoTopicName>
+                <frameName>${prefix}_camera</frameName>
+                <hackBaseline>0.07</hackBaseline>
+                <distortionK1>0.0</distortionK1>
+                <distortionK2>0.0</distortionK2>
+                <distortionK3>0.0</distortionK3>
+                <distortionT1>0.0</distortionT1>
+                <distortionT2>0.0</distortionT2>
+            </plugin>
+            </sensor>
+        </gazebo>
     </xacro:macro>
 </robot>

File: src/arm_urdf/urdf/arm_urdf.xacro (robot description, xacro)
@@ -4,4 +4,16 @@
         <!-- links -->
         <link name="${prefix}_base_fixed">
+            <visual>
+            <origin rpy="0 0 0" xyz="0 0 0.4"/>
+            <geometry>
+                <box size="0.3 0.5 1"/>
+            </geometry>
+            </visual>
+            <collision>
+            <origin rpy="0 0 0" xyz="0 0 0.4"/>
+            <geometry>
+                <box size="0.3 0.3 0.8"/>
+            </geometry>
+            </collision>
             <inertial>
             <mass value="0.5"/>
@@ -117,8 +129,27 @@
             </inertial>
         </link>
+        <!-- camera link -->
+        <link name="${prefix}_camera">
+            <visual>
+            <origin rpy="0.0 ${radians(180)} 0" xyz="0 0.06 0.043"/>
+            <geometry>
+                <box size="0.05 0.05 0.08"/>
+            </geometry>
+            </visual>
+            <collision>
+            <origin rpy="0.0 ${radians(180)} 0" xyz="0 0.06 0.043"/>
+            <geometry>
+                <box size="0.05 0.05 0.08"/>
+            </geometry>
+            </collision>
+            <inertial>
+            <mass value="0.5"/>
+            <inertia ixx="0.4" ixy="0.0" ixz="0.0" iyy="0.4" iyz="0.0" izz="0.2"/>
+            </inertial>
+        </link>
         <!-- joints -->
-        <!-- joint names defined like so: ${prefix}_<parent>-<child>_joint -->
+        <!-- joint names defined like so: ${prefix}_<parent>_<child>_joint -->
         <joint name="${prefix}_base_fixed_base_joint" type="revolute">
-            <origin rpy="0.0 0 0" xyz="0.0 0 0"/>
+            <origin rpy="0 ${radians(90)} 0" xyz="0.15 0 0.6"/>
             <axis xyz="0 0 1"/>
             <limit effort="1000.0" lower="${radians(-180)}" upper="${radians(180)}" velocity="0.5"/>
@@ -164,4 +195,10 @@
             <dynamics D="1" K="7000" mu_coulomb="0" mu_viscous="16" damping="0.003" friction="0.0"/>
         </joint>
+        <!-- camera joint -->
+        <joint name="${prefix}_wrist_link_camera_joint" type="fixed">
+            <origin rpy="0 0 0" xyz="0 0.0 0"/>
+            <parent link="${prefix}_wrist_link" />
+            <child link="${prefix}_camera" />
+        </joint>
     </xacro:macro>
 </robot>

File: src/arm_urdf/urdf/main.xacro (robot description, xacro)
@@ -1,19 +1,28 @@
 <?xml version="1.0" ?>
 <robot xmlns:xacro="http://www.ros.org/wiki/xacro" name="robot">
-    <!-- include statements, much like import statements -->
+    <!-- ################################################### -->
+    <!-- # include statements, much like import statements -->
+    <!-- ################################################### -->
     <xacro:include filename="$(find arm_urdf)/urdf/arm_urdf.xacro"/>
     <xacro:include filename="$(find arm_urdf)/urdf/arm_gazebo.xacro"/>
     <xacro:include filename="$(find arm_urdf)/urdf/arm_control.xacro"/>
+    <!-- ################################################### -->
+    <!-- # constants -->
+    <!-- ################################################### -->
+    <xacro:property name="arm_prefix" value="arm1" />
+    <!-- ################################################### -->
+    <!-- # Etc -->
+    <!-- ################################################### -->
+    <!-- NOTE: order of execution of xacro does not matter -->
     <!-- name must be kept as "world" for it is a Gazebo keyword for world origin -->
     <link name="world"/>
     <!-- using arm macro defined in arm_urdf.xacro to define robot -->
-    <xacro:arm prefix="arm1"/>
-    <xacro:arm_gazebo_setting prefix="arm1"/>
-    <xacro:arm_control_setting prefix="arm1" />
+    <xacro:arm prefix="${arm_prefix}"/>
+    <xacro:arm_gazebo_setting prefix="${arm_prefix}"/>
+    <xacro:arm_control_setting prefix="${arm_prefix}" />
     <!-- connect the arm to world with fixed joint -->
     <joint name="base" type="fixed">
         <parent link="world" />
-        <child link="arm1_base_fixed" />
+        <child link="${arm_prefix}_base_fixed" />
     </joint>
-    <!-- NOTE: order of execution of above xacro does not matter -->
 </robot>

Commit message: added gripper

File: src/arm_urdf/urdf/arm_control.xacro (robot description, xacro)
@@ -19,4 +19,9 @@
         <xacro:arm_control transmission="${prefix}_tran_3" joint="${prefix}_housing_wrist_link_joint" motor="${prefix}_motor_3"/>
         <xacro:arm_control transmission="${prefix}_tran_4" joint="${prefix}_wrist_link_wrist_cuff_joint" motor="${prefix}_motor_4"/>
+        <xacro:arm_control transmission="${prefix}_tran_5" joint="${prefix}_palm_hub_left_joint" motor="${prefix}_motor_5"/>
+        <xacro:arm_control transmission="${prefix}_tran_6" joint="${prefix}_hub_left_finger_left_joint" motor="${prefix}_motor_6"/>
+        <xacro:arm_control transmission="${prefix}_tran_7" joint="${prefix}_palm_hub_right_joint" motor="${prefix}_motor_7"/>
+        <xacro:arm_control transmission="${prefix}_tran_8" joint="${prefix}_hub_right_finger_right_joint" motor="${prefix}_motor_8"/>
+        <xacro:arm_control transmission="${prefix}_tran_9" joint="${prefix}_palm_finger_thumb_joint" motor="${prefix}_motor_9"/>
     </xacro:macro>
 </robot>

File: src/arm_urdf/urdf/arm_gazebo.xacro (robot description, xacro)
@@ -17,43 +17,46 @@
             <plugin name="gazebo_ros_control" filename="libgazebo_ros_control.so"/>
         </gazebo>
-        <gazebo reference="${prefix}_camera">
-            <sensor type="camera" name="camera1">
-            <update_rate>30.0</update_rate>
-            <camera name="head">
-                <horizontal_fov>1.3962634</horizontal_fov>
+        <!-- camera description adapted from http://gazebosim.org/tutorials?tut=ros_gzplugins#Pluginsavailableingazebo_plugins -->
+        <gazebo reference="${prefix}_camera_link">
+            <sensor name="${prefix}_camera" type="depth">
+                <update_rate>20</update_rate>
+                <camera>
+                <horizontal_fov>1.047198</horizontal_fov>
                 <image>
-                <width>800</width>
-                <height>800</height>
-                <format>R8G8B8</format>
+                    <width>640</width>
+                    <height>480</height>
+                    <format>R8G8B8</format>
                 </image>
                 <clip>
-                <near>0.02</near>
-                <far>300</far>
+                    <near>0.05</near>
+                    <far>3</far>
                 </clip>
-                <noise>
-                <type>gaussian</type>
-                <!-- Noise is sampled independently per pixel on each frame.
-                    That pixel's noise value is added to each of its color
-                    channels, which at that point lie in the range [0,1]. -->
-                <mean>0.0</mean>
-                <stddev>0.007</stddev>
-                </noise>
-            </camera>
-            <plugin name="camera_controller" filename="libgazebo_ros_camera.so">
+                </camera>
+                <plugin name="${prefix}_kinetic_camera_controller" filename="libgazebo_ros_openni_kinect.so">
+                <baseline>0.2</baseline>
                 <alwaysOn>true</alwaysOn>
-                <updateRate>0.0</updateRate>
-                <cameraName>bot/camera1</cameraName>
-                <imageTopicName>image_raw</imageTopicName>
-                <cameraInfoTopicName>camera_info</cameraInfoTopicName>
-                <frameName>${prefix}_camera</frameName>
-                <hackBaseline>0.07</hackBaseline>
-                <distortionK1>0.0</distortionK1>
-                <distortionK2>0.0</distortionK2>
-                <distortionK3>0.0</distortionK3>
-                <distortionT1>0.0</distortionT1>
-                <distortionT2>0.0</distortionT2>
-            </plugin>
+                <updateRate>1.0</updateRate>
+                <cameraName>${prefix}_camera_ir</cameraName>
+                <imageTopicName>/${prefix}_camera/color/image_raw</imageTopicName>
+                <cameraInfoTopicName>/${prefix}_camera/color/camera_info</cameraInfoTopicName>
+                <depthImageTopicName>/${prefix}_camera/depth/image_raw</depthImageTopicName>
+                <depthImageInfoTopicName>/${prefix}_camera/depth/camera_info</depthImageInfoTopicName>
+                <pointCloudTopicName>/${prefix}_camera/depth/points</pointCloudTopicName>
+                <frameName>${prefix}_camera_link</frameName>
+                <pointCloudCutoff>0.5</pointCloudCutoff>
+                <pointCloudCutoffMax>3.0</pointCloudCutoffMax>
+                <distortionK1>0.00000001</distortionK1>
+                <distortionK2>0.00000001</distortionK2>
+                <distortionK3>0.00000001</distortionK3>
+                <distortionT1>0.00000001</distortionT1>
+                <distortionT2>0.00000001</distortionT2>
+                <CxPrime>0</CxPrime>
+                <Cx>0</Cx>
+                <Cy>0</Cy>
+                <focalLength>0</focalLength>
+                <hackBaseline>0</hackBaseline>
+                </plugin>
             </sensor>
-        </gazebo>
+            </gazebo>
     </xacro:macro>
 </robot>

File: src/arm_urdf/urdf/arm_urdf.xacro (robot description, xacro)
@@ -1,4 +1,6 @@
 <?xml version="1.0"?>
 <robot xmlns:xacro="http://www.ros.org/wiki/xacro" name="robot">
+    <!-- import  -->
+    <xacro:include filename="$(find arm_urdf)/urdf/gripper_urdf.xacro"/>
     <xacro:macro name="arm" params="prefix">
         <!-- links -->
@@ -130,22 +132,24 @@
         </link>
         <!-- camera link -->
-        <link name="${prefix}_camera">
-            <visual>
-            <origin rpy="0.0 ${radians(180)} 0" xyz="0 0.06 0.043"/>
-            <geometry>
-                <box size="0.05 0.05 0.08"/>
-            </geometry>
-            </visual>
-            <collision>
-            <origin rpy="0.0 ${radians(180)} 0" xyz="0 0.06 0.043"/>
-            <geometry>
-                <box size="0.05 0.05 0.08"/>
-            </geometry>
-            </collision>
-            <inertial>
-            <mass value="0.5"/>
-            <inertia ixx="0.4" ixy="0.0" ixz="0.0" iyy="0.4" iyz="0.0" izz="0.2"/>
-            </inertial>
-        </link>
+        <link name="${prefix}_camera_link">
+            <visual>
+            <origin rpy="0.0 ${radians(180)} 0" xyz="0 0 0"/>
+            <geometry>
+                <box size="0.08 0.05 0.05"/>
+            </geometry>
+            </visual>
+            <collision>
+            <origin rpy="0.0 ${radians(180)} 0" xyz="0 0 0"/>
+            <geometry>
+                <box size="0.08 0.05 0.05"/>
+            </geometry>
+            </collision>
+            <inertial>
+            <mass value="0.5"/>
+            <inertia ixx="0.4" ixy="0.0" ixz="0.0" iyy="0.4" iyz="0.0" izz="0.2"/>
+            </inertial>
+        </link>
+        <!-- gripper -->
+        <xacro:gripper prefix="${prefix}"/>
         <!-- joints -->
         <!-- joint names defined like so: ${prefix}_<parent>_<child>_joint -->
@@ -196,8 +200,14 @@
         </joint>
         <!-- camera joint -->
-        <joint name="${prefix}_wrist_link_camera_joint" type="fixed">
-            <origin rpy="0 0 0" xyz="0 0.0 0"/>
-            <parent link="${prefix}_wrist_link" />
-            <child link="${prefix}_camera" />
+        <joint name="${prefix}_base_fixed_camera_link_joint" type="fixed">
+            <origin rpy="0 0 0" xyz="0.2 0 0.3"/>
+            <parent link="${prefix}_base_fixed" />
+            <child link="${prefix}_camera_link" />
+        </joint>
+        <!-- gripper joint  -->
+        <joint name="${prefix}_wrist_cuff_palm_joint" type="fixed">
+            <origin rpy="0 0 0" xyz="0 0.0 0.03"/>
+            <parent link="${prefix}_wrist_cuff" />
+            <child link="${prefix}_palm" />
         </joint>
     </xacro:macro>

File: src/arm_urdf/urdf/gripper_only.xacro (robot description, xacro)
@@ -4,11 +4,9 @@
     <!-- # include statements, much like import statements -->
     <!-- ################################################### -->
-    <xacro:include filename="$(find arm_urdf)/urdf/arm_urdf.xacro"/>
-    <xacro:include filename="$(find arm_urdf)/urdf/arm_gazebo.xacro"/>
-    <xacro:include filename="$(find arm_urdf)/urdf/arm_control.xacro"/>
+    <xacro:include filename="$(find arm_urdf)/urdf/gripper_urdf.xacro"/>
     <!-- ################################################### -->
     <!-- # constants -->
     <!-- ################################################### -->
-    <xacro:property name="arm_prefix" value="arm1" />
+    <xacro:property name="gripper_prefix" value="gripper1" />
     <!-- ################################################### -->
     <!-- # Etc -->
@@ -17,12 +15,10 @@
     <!-- name must be kept as "world" for it is a Gazebo keyword for world origin -->
     <link name="world"/>
-    <!-- using arm macro defined in arm_urdf.xacro to define robot -->
-    <xacro:arm prefix="${arm_prefix}"/>
-    <xacro:arm_gazebo_setting prefix="${arm_prefix}"/>
-    <xacro:arm_control_setting prefix="${arm_prefix}" />
+    <!-- using gripper macro defined in gripper_urdf.xacro to define robot -->
+    <xacro:gripper prefix="${gripper_prefix}"/>
     <!-- connect the arm to world with fixed joint -->
     <joint name="base" type="fixed">
         <parent link="world" />
-        <child link="${arm_prefix}_base_fixed" />
+        <child link="${gripper_prefix}_palm" />
     </joint>
 </robot>
