Commit message: base camera

File: src/arm_urdf/urdf/arm_gazebo.xacro (robot description, xacro)
@@ -2,4 +2,7 @@
 <robot xmlns:xacro="http://www.ros.org/wiki/xacro">
     <xacro:macro name="arm_gazebo_setting" params="prefix">
+    <xacro:property name="camera_link" value="arm_base_camera" />
+    <xacro:property name="camera_name" value="kinect" />
+    <xacro:property name="frame_name" value="kinect_frame" />
         <xacro:macro name="arm_gazebo" params="link">
             <gazebo reference="${link}">
@@ -14,5 +17,46 @@
         <xacro:arm_gazebo link="${prefix}_wrist_link"/>
         <xacro:arm_gazebo link="${prefix}_wrist_cuff"/>
-        <gazebo>
+        <gazebo reference="${camera_link}">
+            <sensor name="${camera_link}_camera" type="depth">
+                <update_rate>20</update_rate>
+                <camera>
+                <horizontal_fov>1.047198</horizontal_fov>
+                <image>
+                    <width>640</width>
+                    <height>480</height>
+                    <format>R8G8B8</format>
+                </image>
+                <clip>
+                    <near>0.05</near>
+                    <far>3</far>
+                </clip>
+                </camera>
+                <plugin name="${camera_link}_controller" filename="libgazebo_ros_openni_kinect.so">
+                <baseline>0.2</baseline>
+                <alwaysOn>true</alwaysOn>
+                <updateRate>1.0</updateRate>
+                <cameraName>${camera_name}_ir</cameraName>
+                <imageTopicName>/${camera_name}/color/image_raw</imageTopicName>
+                <cameraInfoTopicName>/${camera_name}/color/camera_info</cameraInfoTopicName>
+                <depthImageTopicName>/${camera_name}/depth/image_raw</depthImageTopicName>
+                <depthImageInfoTopicName>/${camera_name}/depth/camera_info</depthImageInfoTopicName>
+                <pointCloudTopicName>/${camera_name}/depth/points</pointCloudTopicName>
+                <frameName>${frame_name}</frameName>
+                <pointCloudCutoff>0.5</pointCloudCutoff>
+                <pointCloudCutoffMax>3.0</pointCloudCutoffMax>
+                <distortionK1>0.00000001</distortionK1>
+                <distortionK2>0.00000001</distortionK2>
+                <distortionK3>0.00000001</distortionK3>
+                <distortionT1>0.00000001</distortionT1>
+                <distortionT2>0.00000001</distortionT2>
+                <CxPrime>0</CxPrime>
+                <Cx>0</Cx>
+                <Cy>0</Cy>
+                <focalLength>0</focalLength>
+                <hackBaseline>0</hackBaseline>
+                </plugin>
+            </sensor>
+        </gazebo>
+        <!-- <gazebo>
             <plugin name="gazebo_ros_control" filename="libgazebo_ros_control.so"/>
         </gazebo>
@@ -33,7 +77,4 @@
                 <noise>
                 <type>gaussian</type>
-                <!-- Noise is sampled independently per pixel on each frame.
-                    That pixel's noise value is added to each of its color
-                    channels, which at that point lie in the range [0,1]. -->
                 <mean>0.0</mean>
                 <stddev>0.007</stddev>
@@ -55,5 +96,5 @@
             </plugin>
             </sensor>
-        </gazebo>
+        </gazebo> -->
     </xacro:macro>
 </robot>

File: src/arm_urdf/urdf/arm_urdf.xacro (robot description, xacro)
@@ -130,5 +130,5 @@
         </link>
         <!-- camera link -->
-        <link name="${prefix}_camera">
+        <link name="${prefix}_base_camera">
             <visual>
             <origin rpy="0.0 ${radians(180)} 0" xyz="0 0.06 0.043"/>
@@ -196,8 +196,8 @@
         </joint>
         <!-- camera joint -->
-        <joint name="${prefix}_wrist_link_camera_joint" type="fixed">
-            <origin rpy="0 0 0" xyz="0 0.0 0"/>
-            <parent link="${prefix}_wrist_link" />
-            <child link="${prefix}_camera" />
+        <joint name="${prefix}_base_camera_joint" type="fixed">
+            <origin rpy="0 ${pi/2} 0" xyz="0.15 0 0.8"/>
+            <parent link="${prefix}_base_fixed" />
+            <child link="${prefix}_base_camera" />
         </joint>
     </xacro:macro>

Commit message: added camera to base pedestal

File: src/arm_urdf/urdf/arm_gazebo.xacro (robot description, xacro)
@@ -2,7 +2,4 @@
 <robot xmlns:xacro="http://www.ros.org/wiki/xacro">
     <xacro:macro name="arm_gazebo_setting" params="prefix">
-    <xacro:property name="camera_link" value="arm_base_camera" />
-    <xacro:property name="camera_name" value="kinect" />
-    <xacro:property name="frame_name" value="kinect_frame" />
         <xacro:macro name="arm_gazebo" params="link">
             <gazebo reference="${link}">
@@ -17,44 +14,44 @@
         <xacro:arm_gazebo link="${prefix}_wrist_link"/>
         <xacro:arm_gazebo link="${prefix}_wrist_cuff"/>
-        <gazebo reference="${camera_link}">
-            <sensor name="${camera_link}_camera" type="depth">
-                <update_rate>20</update_rate>
-                <camera>
-                <horizontal_fov>1.047198</horizontal_fov>
-                <image>
-                    <width>640</width>
-                    <height>480</height>
-                    <format>R8G8B8</format>
-                </image>
-                <clip>
-                    <near>0.05</near>
-                    <far>3</far>
-                </clip>
-                </camera>
-                <plugin name="${camera_link}_controller" filename="libgazebo_ros_openni_kinect.so">
-                <baseline>0.2</baseline>
-                <alwaysOn>true</alwaysOn>
-                <updateRate>1.0</updateRate>
-                <cameraName>${camera_name}_ir</cameraName>
-                <imageTopicName>/${camera_name}/color/image_raw</imageTopicName>
-                <cameraInfoTopicName>/${camera_name}/color/camera_info</cameraInfoTopicName>
-                <depthImageTopicName>/${camera_name}/depth/image_raw</depthImageTopicName>
-                <depthImageInfoTopicName>/${camera_name}/depth/camera_info</depthImageInfoTopicName>
-                <pointCloudTopicName>/${camera_name}/depth/points</pointCloudTopicName>
-                <frameName>${frame_name}</frameName>
-                <pointCloudCutoff>0.5</pointCloudCutoff>
-                <pointCloudCutoffMax>3.0</pointCloudCutoffMax>
-                <distortionK1>0.00000001</distortionK1>
-                <distortionK2>0.00000001</distortionK2>
-                <distortionK3>0.00000001</distortionK3>
-                <distortionT1>0.00000001</distortionT1>
-                <distortionT2>0.00000001</distortionT2>
-                <CxPrime>0</CxPrime>
-                <Cx>0</Cx>
-                <Cy>0</Cy>
-                <focalLength>0</focalLength>
-                <hackBaseline>0</hackBaseline>
-                </plugin>
-            </sensor>
+        <gazebo reference="${camera_link_name}">
+        <sensor name="${camera_link_name}_camera" type="depth">
+            <update_rate>20</update_rate>
+            <camera>
+            <horizontal_fov>1.047198</horizontal_fov>
+            <image>
+                <width>640</width>
+                <height>480</height>
+                <format>R8G8B8</format>
+            </image>
+            <clip>
+                <near>0.05</near>
+                <far>3</far>
+            </clip>
+            </camera>
+            <plugin name="${camera_link_name}_controller" filename="libgazebo_ros_openni_kinect.so">
+            <baseline>0.2</baseline>
+            <alwaysOn>true</alwaysOn>
+            <updateRate>1.0</updateRate>
+            <cameraName>${camera_name}_ir</cameraName>
+            <imageTopicName>/${camera_name}/color/image_raw</imageTopicName>
+            <cameraInfoTopicName>/${camera_name}/color/camera_info</cameraInfoTopicName>
+            <depthImageTopicName>/${camera_name}/depth/image_raw</depthImageTopicName>
+            <depthImageInfoTopicName>/${camera_name}/depth/camera_info</depthImageInfoTopicName>
+            <pointCloudTopicName>/${camera_name}/depth/points</pointCloudTopicName>
+            <frameName>${frame_name}</frameName>
+            <pointCloudCutoff>0.5</pointCloudCutoff>
+            <pointCloudCutoffMax>3.0</pointCloudCutoffMax>
+            <distortionK1>0.00000001</distortionK1>
+            <distortionK2>0.00000001</distortionK2>
+            <distortionK3>0.00000001</distortionK3>
+            <distortionT1>0.00000001</distortionT1>
+            <distortionT2>0.00000001</distortionT2>
+            <CxPrime>0</CxPrime>
+            <Cx>0</Cx>
+            <Cy>0</Cy>
+            <focalLength>0</focalLength>
+            <hackBaseline>0</hackBaseline>
+            </plugin>
+        </sensor>
         </gazebo>
         <!-- <gazebo>

File: src/arm_urdf/urdf/arm_urdf.xacro (robot description, xacro)
@@ -1,4 +1,8 @@
 <?xml version="1.0"?>
 <robot xmlns:xacro="http://www.ros.org/wiki/xacro" name="robot">
+    <xacro:property name="camera_link_name" value="arm_base_camera" />
+    <xacro:property name="camera_name" value="kinect"/>
+    <xacro:property name="frame_name" value="kinect_frame"/>
+    <xacro:property name="view_angle" value="30" />
     <xacro:macro name="arm" params="prefix">
         <!-- links -->
@@ -122,23 +126,4 @@
             <geometry>
                 <mesh filename="package://arm_urdf/meshes/Wrist Cuff.dae"/>
-            </geometry>
-            </collision>
-            <inertial>
-            <mass value="0.5"/>
-            <inertia ixx="0.4" ixy="0.0" ixz="0.0" iyy="0.4" iyz="0.0" izz="0.2"/>
-            </inertial>
-        </link>
-        <!-- camera link -->
-        <link name="${prefix}_base_camera">
-            <visual>
-            <origin rpy="0.0 ${radians(180)} 0" xyz="0 0.06 0.043"/>
-            <geometry>
-                <box size="0.05 0.05 0.08"/>
-            </geometry>
-            </visual>
-            <collision>
-            <origin rpy="0.0 ${radians(180)} 0" xyz="0 0.06 0.043"/>
-            <geometry>
-                <box size="0.05 0.05 0.08"/>
             </geometry>
             </collision>
@@ -195,9 +180,29 @@
             <dynamics D="1" K="7000" mu_coulomb="0" mu_viscous="16" damping="0.003" friction="0.0"/>
         </joint>
+        <!-- camera -->
+        <!-- camera link -->
+        <link name="arm_base_camera">
+            <visual>
+            <origin rpy="0.0 ${radians(180)} 0" xyz="0 0.06 0.043"/>
+            <geometry>
+                <box size="0.05 0.05 0.08"/>
+            </geometry>
+            </visual>
+            <collision>
+            <origin rpy="0.0 ${radians(180)} 0" xyz="0 0.06 0.043"/>
+            <geometry>
+                <box size="0.05 0.05 0.08"/>
+            </geometry>
+            </collision>
+            <inertial>
+            <mass value="0.5"/>
+            <inertia ixx="0.4" ixy="0.0" ixz="0.0" iyy="0.4" iyz="0.0" izz="0.2"/>
+            </inertial>
+        </link>
         <!-- camera joint -->
-        <joint name="${prefix}_base_camera_joint" type="fixed">
-            <origin rpy="0 ${pi/2} 0" xyz="0.15 0 0.8"/>
+        <joint name="arm_base_camera_joint" type="fixed">
+            <origin rpy="0 ${radians(view_angle)} 0" xyz="0.15 0 0.8"/>
             <parent link="${prefix}_base_fixed" />
-            <child link="${prefix}_base_camera" />
+            <child link="arm_base_camera" />
         </joint>
     </xacro:macro>

Commit message: fixed broken merge

File: src/arm_urdf/urdf/arm_gazebo.xacro (robot description, xacro)
@@ -2,7 +2,4 @@
 <robot xmlns:xacro="http://www.ros.org/wiki/xacro">
     <xacro:macro name="arm_gazebo_setting" params="prefix">
-    <xacro:property name="camera_link" value="arm_base_camera" />
-    <xacro:property name="camera_name" value="kinect" />
-    <xacro:property name="frame_name" value="kinect_frame" />
         <xacro:macro name="arm_gazebo" params="link">
             <gazebo reference="${link}">
@@ -17,6 +14,10 @@
         <xacro:arm_gazebo link="${prefix}_wrist_link"/>
         <xacro:arm_gazebo link="${prefix}_wrist_cuff"/>
-        <gazebo reference="${camera_link}">
-            <sensor name="${camera_link}_camera" type="depth">
+        <gazebo>
+            <plugin name="gazebo_ros_control" filename="libgazebo_ros_control.so"/>
+        </gazebo>
+        <!-- camera description adapted from http://gazebosim.org/tutorials?tut=ros_gzplugins#Pluginsavailableingazebo_plugins -->
+        <gazebo reference="${prefix}_camera_link">
+            <sensor name="${prefix}_camera" type="depth">
                 <update_rate>20</update_rate>
                 <camera>
@@ -32,15 +33,15 @@
                 </clip>
                 </camera>
-                <plugin name="${camera_link}_controller" filename="libgazebo_ros_openni_kinect.so">
+                <plugin name="${prefix}_kinetic_camera_controller" filename="libgazebo_ros_openni_kinect.so">
                 <baseline>0.2</baseline>
                 <alwaysOn>true</alwaysOn>
                 <updateRate>1.0</updateRate>
-                <cameraName>${camera_name}_ir</cameraName>
-                <imageTopicName>/${camera_name}/color/image_raw</imageTopicName>
-                <cameraInfoTopicName>/${camera_name}/color/camera_info</cameraInfoTopicName>
-                <depthImageTopicName>/${camera_name}/depth/image_raw</depthImageTopicName>
-                <depthImageInfoTopicName>/${camera_name}/depth/camera_info</depthImageInfoTopicName>
-                <pointCloudTopicName>/${camera_name}/depth/points</pointCloudTopicName>
-                <frameName>${frame_name}</frameName>
+                <cameraName>${prefix}_camera_ir</cameraName>
+                <imageTopicName>/${prefix}_camera/color/image_raw</imageTopicName>
+                <cameraInfoTopicName>/${prefix}_camera/color/camera_info</cameraInfoTopicName>
+                <depthImageTopicName>/${prefix}_camera/depth/image_raw</depthImageTopicName>
+                <depthImageInfoTopicName>/${prefix}_camera/depth/camera_info</depthImageInfoTopicName>
+                <pointCloudTopicName>/${prefix}_camera/depth/points</pointCloudTopicName>
+                <frameName>${prefix}_camera_link</frameName>
                 <pointCloudCutoff>0.5</pointCloudCutoff>
                 <pointCloudCutoffMax>3.0</pointCloudCutoffMax>
@@ -57,5 +58,5 @@
                 </plugin>
             </sensor>
-        </gazebo>
+            </gazebo>
     </xacro:macro>
 </robot>
