Commit message: + gitignore, + gazebo_worlds pkg

File: src/arm_urdf/urdf/arm_urdf.xacro (robot description, xacro)
@@ -157,5 +157,5 @@
             <origin rpy="0 ${radians(90)} 0" xyz="0.15 0 0.6"/>
             <axis xyz="0 0 1"/>
-            <limit effort="1000.0" lower="${radians(-180)}" upper="${radians(180)}" velocity="0.5"/>
+            <limit effort="1000.0" lower="${radians(-180)}" upper="${radians(180)}" velocity="2.5"/>
             <parent link="${prefix}_base_fixed" />
             <child link="${prefix}_base" />
@@ -165,5 +165,5 @@
             <origin rpy="0.0 0 0" xyz="0.0 0 0.165"/>
             <axis xyz="1 0 0"/>
-            <limit effort="1000.0" lower="${radians(-120)}" upper="${radians(120)}" velocity="0.5"/>
+            <limit effort="1000.0" lower="${radians(-120)}" upper="${radians(120)}" velocity="2.5"/>
             <parent link="${prefix}_base" />
             <child link="${prefix}_bridge" />
@@ -178,5 +178,5 @@
             <origin rpy="0 0 0" xyz="0 0 0.24875"/>
             <axis xyz="1 0 0"/>
-            <limit effort="1000.0" lower="${radians(-165)}" upper="${radians(165)}" velocity="0.5"/>
+            <limit effort="1000.0" lower="${radians(-165)}" upper="${radians(165)}" velocity="2.5"/>
             <parent link="${prefix}_bridge" />
             <child link="${prefix}_housing" />
@@ -186,5 +186,5 @@
             <origin rpy="0 0 0" xyz="0 0 0.045"/>
             <axis xyz="0 0 1"/>
-            <limit effort="1000.0" lower="${radians(-180)}" upper="${radians(180)}" velocity="0.5"/>
+            <limit effort="1000.0" lower="${radians(-180)}" upper="${radians(180)}" velocity="2.5"/>
             <parent link="${prefix}_housing" />
             <child link="${prefix}_wrist_link" />
@@ -194,5 +194,5 @@
             <origin rpy="0 0 0" xyz="0 0.0 0.122"/>
             <axis xyz="1 0 0"/>
-            <limit effort="1000.0" lower="${radians(-85)}" upper="${radians(85)}" velocity="0.5"/>
+            <limit effort="1000.0" lower="${radians(-85)}" upper="${radians(85)}" velocity="2.5"/>
             <parent link="${prefix}_wrist_link" />
             <child link="${prefix}_wrist_cuff" />
